File: HTMDv2.2s.kicad_sch (KiCad schematic)
At the start: 72 parts, among them IC1 TJA1441AT_0Z, IC2 A3921KLPTR-T, J1 Conn_01x04, J2 Conn_01x04, J3 Conn_01x06, J4 Conn_01x01, J5 Conn_01x01_Pin, J6 Conn_01x02_Pin, J7 Conn_01x01_Pin, J8 Conn_01x01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

Commit message: update
Parts:
- removed D14: RB160M-30TR, Diode_SMD:D_SOD-123, symbol YamaMotherV4-rescue:RB160M-30TR-diode
- removed U3: ADUM140E0BRWZ-RL, 0-Myparts:ADuM140E, symbol 0-Myparts:ADUM140E0BRWZ-RL
- added C9: C, symbol Device:C
- added D4: D, 0-Myparts:SS2040FL, symbol Device:D
- added U3: ISO6741FDWR, 0_Mylib:ISO674x, symbol 0_symbols:ISO6741FDWR
- added U4: CZ3A07, 0_Mylib:CZ3A07, symbol 0_symbols:CZ3A07
- J6: footprint (none) -> Connector_PinHeader_2.54mm:PinHeader_1x02_P2.54mm_Horizontal
- J9: footprint (none) -> Connector_PinHeader_2.54mm:PinHeader_1x04_P2.54mm_Horizontal
- R16, R17: footprint (none) -> Resistor_SMD:R_0603_1608Metric_Pad0.98x0.95mm_HandSolder
Connections:
- net +3.3V: now also C9.1, U3.1 (VCC1), U3.7 (EN1), U4.13 (VDD)
- net +3V3: now also D4.2 (A)
- net +5VA: now also U3.10 (EN2), U3.16 (VCC2)
- net GND: now also C9.2, U3.2 (GND1), U3.8 (GND1), U4.16 (VSS_2), U4.9 (VSS_1)
- net GNDPWR: now also U3.15 (GND2), U3.9 (GND2)
- net OPHASE1: now also U3.3 (INA)
- net OPWMH1: now also U3.6 (OUTD)
- net OPWML1: now also U3.5 (OUTC)
- net OSR1: now also U3.4 (INB)
- net PHASE1: now also U3.14 (OUTA)
- net PWMH1: now also U3.11 (IND)
- net PWML1: now also U3.12 (INC)
- net SR1: now also U3.13 (OUTB)
- net at J9.4 (Pin_4): now also D4.1 (K)
- net SA1 renamed IP
- net IP: now also U4.1 (IP); no longer J4.1 (Pin_1)
- new net IN: J4.1 (Pin_1), U4.5 (IN)
- new net OCD1: U4.11 (OCD2)
- new net OCD2: U4.10 (OCD1)
- new net VOUT: U4.12 (VOUT)
- new net VREF1: U4.14 (REF1)
- new net VREF2: U4.15 (REF2)
- no-connect marks 5 -> 3
Other:
- note added: "all 20kohm"
- note added: "通信用インターフェース"
- moved on the sheet: C7, C8, R4, R5, R6, R9

Commit message: Update HTMDv2.2s.kicad_sch
Parts:
- removed C4: 0.1u, Capacitor_SMD:C_0603_1608Metric_Pad1.08x0.95mm_HandSolder, symbol Device:C
- removed C5: 10u, Capacitor_SMD:C_0805_2012Metric, symbol Device:C
- removed D4: D, 0-Myparts:SS2040FL, symbol Device:D
- removed R17: 10k, Resistor_SMD:R_0603_1608Metric_Pad0.98x0.95mm_HandSolder, symbol Device:R
- removed SW1: SW_Push, 0-Myparts:TVAF06, symbol Switch:SW_Push
- removed U2: STM32F303K8Tx, Package_QFP:LQFP-32_7x7mm_P0.8mm, symbol MCU_ST_STM32F3:STM32F303K8Tx
- added C10, C11, C17, C18: 0.1u, symbol Device:C
- added C12: 4.7u, symbol Device:C
- added C15: 10u, symbol Device:C
- added J10, J11: Conn_01x02, symbol Connector_Generic:Conn_01x02
- added R26, R27: 1k, symbol Device:R
- added R28, R29: 10k, symbol Device:R
- added U2: STM32G431CBUx, Package_DFN_QFN:QFN-48-1EP_7x7mm_P0.5mm_EP5.6x5.6mm, symbol MCU_ST_STM32G4:STM32G431CBUx
- added U5: MCP3421A0T-ECH, symbol Analog_ADC:MCP3421A0T-ECH
- C6: value 0.1u -> 1n; footprint Capacitor_SMD:C_0603_1608Metric_Pad1.08x0.95mm_HandSolder -> (none)
- R1, R8: value 10k -> 20k; footprint Resistor_SMD:R_0603_1608Metric -> (none)
Connections:
- net +3.3V: now also C10.1, C11.1, C12.1, C18.1, J10.2 (Pin_2), J11.2 (Pin_2), U2.1 (VBAT), U2.20 (VREF+), U2.21 (VDDA), U2.23 (VDD), U2.35 (VDD), U2.48 (VDD); no longer R1.1, R8.1
- net +3V3: now also J9.4 (Pin_4)
- net CAN_RX: now also U2.33 (PA11)
- net CAN_TX: now also U2.34 (PA12)
- net ENC_A: now also U2.30 (PA8)
- net ENC_B: now also U2.31 (PA9)
- net GND: now also R1.2, R8.2, C10.2, C11.2, C12.2, C15.2, C17.2, C18.2, U2.46 (PB8), U2.49 (VSS), U5.2 (Vss); no longer C6.2
- net I2C_SCL: now also R28.2, U2.38 (PA15), U5.3 (SCL)
- net I2C_SDA: now also R29.2, U2.45 (PB7), U5.4 (SDA)
- net LED1: now also U2.29 (PC6)
- net LED2: now also U2.28 (PB15)
- net LED3: now also U2.27 (PB14)
- net LED4: now also U2.26 (PB13)
- net LED5: now also U2.25 (PB12)
- net OCD1: now also U2.3 (PC14)
- net OCD2: now also U2.4 (PC15)
- net OPHASE1: now also U2.11 (PA3)
- net OPWMH1: now also U2.8 (PA0)
- net OPWML1: now also U2.9 (PA1)
- net OSR1: now also U2.10 (PA2)
- net SPI_MISO: now also U2.14 (PA6)
- net SPI_MOSI: now also U2.15 (PA7)
- net SPI_SCK: now also U2.13 (PA5)
- net SWCLK: now also U2.37 (PA14)
- net SWDIO: now also U2.36 (PA13)
- net UART_RX: now also U2.40 (PC11)
- net UART_TX: now also U2.39 (PC10)
- net VCC: now also C15.1, C17.1, R28.1, R29.1, U5.5 (Vdd)
- net BOOT: no longer names the net of C6.1
- net BOOT: now also R26.2, R27.2, U5.1 (Vin+); no longer R1.2
- net EN renamed NRST
- net NRST: now also U2.7 (PG10); no longer R8.2
- net VOUT: no longer names the net of U4.12 (VOUT)
- net VOUT: now also R26.1
- new net: C6.2, R27.1, U5.6 (Vin-)
- new net LED_CAN: U2.32 (PA10)
- new net LED_LIM1: U2.44 (PB6)
- new net LED_LIM2: U2.41 (PB3)
- new net LIM1: J10.1 (Pin_1), R1.1, U2.47 (PB9)
- new net LIM2: J11.1 (Pin_1), R8.1, U2.43 (PB5)
- new net SPI_CS: U2.16 (PC4)
- no-connect marks 3 -> 13
Other:
- note added: "電流センサ"
- note removed: "BOOTSW"
- note removed: "起動遅延"
- moved on the sheet: C1, C13, C14, C16, C19, C2, C20, C21, C22, C23, C26, C27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

Commit message: Update HTMDv2.2s.kicad_sch
Parts:
- removed D2, D3: LED, LED_SMD:LED_0603_1608Metric_Pad1.05x0.95mm_HandSolder, symbol Device:LED
- added C4, C5: 1n, symbol Device:C
- added IC3: TMP275AQDGKRQ1, 0_Mylib:SOP65P490X110-8N, symbol 0_symbols:TMP275AQDGKRQ1
- added JP1: Jumper_2_Open, TestPoint:TestPoint_2Pads_Pitch2.54mm_Drill0.8mm, symbol Jumper:Jumper_2_Open
- added R17, R30: 10k, symbol Device:R
- added R31: 13k, symbol Device:R
- added R32: 2.4k, symbol Device:R
- added RV1, RV2: 10k, symbol Device:R_Potentiometer_Trim_US
- C7, C8: value C -> 0.1u
- IC1: footprint 0-Myparts:SOIC127P600X175-8N -> SOIC127P600X175-8N
- R2: value R -> 13k; footprint Resistor_SMD:R_0603_1608Metric_Pad0.98x0.95mm_HandSolder -> (none)
- R3: value R -> 2.4k; footprint Resistor_SMD:R_0603_1608Metric_Pad0.98x0.95mm_HandSolder -> (none)
- U1: footprint 0-Myparts:SOT230P700X180-4N -> SOT230P700X180-4N
- U3: footprint 0_Mylib:ISO674x -> SOIC08_7P5X10P3_TEX
Connections:
- net +3V3 is gone; now on net +3.3V: J9.4 (Pin_4)
- net CANRX is gone; now on net CAN_RX: IC1.4 (RXD)
- net CANTX is gone; now on net CAN_TX: IC1.1 (TXD)
- net CLK is gone; now on net SPI_SCK: J3.5 (Pin_5)
- net CS is gone; now on net SPI_CS: J3.6 (Pin_6)
- net MISO is gone; now on net SPI_MISO: J3.3 (Pin_3)
- net MOSI is gone; now on net SPI_MOSI: J3.1 (Pin_1)
- net +3.3V: now also R2.1, IC3.8 (V+), R31.1
- net CANL: now also JP1.2 (B); no longer R10.2
- net GND: now also R3.2, C4.2, C5.2, IC3.4 (GND), IC3.5 (A2), IC3.6 (A1), IC3.7 (A0), R32.2
- net I2C_SCL: now also IC3.1 (SDA), R17.2
- net I2C_SDA: now also IC3.2 (SCL), R30.2
- net LED1: no longer R3.2
- net LED2: no longer R2.2
- net VCC: now also R17.1, R30.1
- net VREF1: now also C4.1, RV1.2
- net VREF2: now also C5.1, RV2.2
- net at R3.1: now also RV1.3
- new net: JP1.1 (A), R10.2
- new net: R2.2, RV1.1
- new net: R31.2, RV2.1
- new net: R32.1, RV2.3
- no-connect marks 13 -> 14
Other:
- note added: "ホール"
- note added: "温度センサ"
- moved on the sheet: C13, C14, C20, C21, C22, C23, C26, C27, C7, C8, H1, H2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

Commit message: Update HTMDv2.2s.kicad_sch
Parts:
- added JP2, JP3, JP4, JP5: SolderJumper_2_Open, Jumper:SolderJumper-2_P1.3mm_Open_TrianglePad1.0x1.5mm, symbol Jumper:SolderJumper_2_Open
- C10, C11, C12, C17, C18, C4, C5, C6, C9: footprint (none) -> Capacitor_SMD:C_0603_1608Metric_Pad1.08x0.95mm_HandSolder
- C15: footprint (none) -> Capacitor_SMD:C_0805_2012Metric_Pad1.18x1.45mm_HandSolder
- IC1: footprint SOIC127P600X175-8N -> (none)
- J10, J11: footprint (none) -> Connector_JST:JST_XH_S2B-XH-A_1x02_P2.50mm_Horizontal
- R1, R17, R2, R26, R27, R28, R29, R3, R30, R31, R32, R8, RV1, RV2: footprint (none) -> Resistor_SMD:R_0603_1608Metric_Pad0.98x0.95mm_HandSolder
- U1: footprint SOT230P700X180-4N -> (none)
- U3: footprint SOIC08_7P5X10P3_TEX -> (none)
Connections:
- net ENC_A: now also JP4.2 (B)
- net ENC_B: now also JP2.2 (B)
- net SPI_MISO: now also JP3.2 (B); no longer J3.3 (Pin_3)
- net SPI_MOSI: now also JP5.2 (B); no longer J3.1 (Pin_1)
- new net: J3.3 (Pin_3), JP2.1 (A), JP3.1 (A)
- new net: J3.1 (Pin_1), JP4.1 (A), JP5.1 (A)

Commit message: update
Parts:
- U3: footprint (none) -> 0_Mylib:ISO674x
- U5: footprint (none) -> Package_TO_SOT_SMD:SOT-23-6_Handsoldering
Other:
- moved on the sheet: J1, J10, J11, J2, J3, JP2, JP3, JP4, JP5, R1, R8

Commit message: update PCB
Parts:
- IC1: footprint (none) -> 0-Myparts:SOIC127P600X175-8N
- IC3: footprint 0_Mylib:SOP65P490X110-8N -> 0_Mylib:TMP275AQDGKRQ1
- RV1, RV2: footprint Resistor_SMD:R_0603_1608Metric_Pad0.98x0.95mm_HandSolder -> 0-Myparts:TSR-3296
- U1: footprint (none) -> 0-Myparts:SOT230P700X180-4N
- U4: footprint 0_Mylib:CZ3A07 -> 0-Myparts:CZ3AG6
Changed lines of the file:
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@@
       (effects (font (size 1.27 1.27)) (justify right))
     )
-    (property "Footprint" "Resistor_SMD:R_0603_1608Metric_Pad0.98x0.95mm_HandSolder" (at 284.226 195.326 0)
+    (property "Footprint" "0-Myparts:TSR-3296" (at 284.226 195.326 0)
       (effects (font (size 1.27 1.27)) hide)
     )
@@
       (effects (font (size 1.27 1.27)))
     )
-    (property "Footprint" "" (at 102.235 41.783 0)
+    (property "Footprint" "0-Myparts:SOT230P700X180-4N" (at 102.235 41.783 0)
       (effects (font (size 1.27 1.27)) (justify bottom) hide)
     )
@@
       (effects (font (size 1.27 1.27)))
     )
-    (property "Footprint" "0_Mylib:SOP65P490X110-8N" (at 286.258 352.349 0)
+    (property "Footprint" "0_Mylib:TMP275AQDGKRQ1" (at 286.258 352.349 0)
       (effects (font (size 1.27 1.27)) (justify left top) hide)
     )
@@
       (effects (font (size 1.27 1.27)))
     )
-    (property "Footprint" "" (at 68.961 244.094 0)
+    (property "Footprint" "0-Myparts:SOIC127P600X175-8N" (at 68.961 244.094 0)
       (effects (font (size 1.27 1.27)) (justify left) hide)
     )
@@
       (effects (font (size 1.27 1.27)) (justify right))
     )
-    (property "Footprint" "Resistor_SMD:R_0603_1608Metric_Pad0.98x0.95mm_HandSolder" (at 312.42 195.199 0)
+    (property "Footprint" "0-Myparts:TSR-3296" (at 312.42 195.199 0)
       (effects (font (size 1.27 1.27)) hide)
     )
@@
       (effects (font (size 1.27 1.27)))
     )
-    (property "Footprint" "0_Mylib:CZ3A07" (at 197.612 283.769 0)
+    (property "Footprint" "0-Myparts:CZ3AG6" (at 197.612 283.769 0)
       (effects (font (size 1.27 1.27)) (justify left top) hide)
     )
@@
   )
   (symbol (lib_id "Analog_ADC:MCP3421A0T-ECH") (at 233.553 200.279 0) (unit 1)
-    (in_bom yes) (on_board yes) (dnp no) (fields_autoplaced)
+    (in_bom yes) (on_board yes) (dnp no)
     (property "Reference" "U5" (at 235.7471 189.23 0)
       (effects (font (size 1.27 1.27)) (justify left))

Commit message: update
Other:
- moved on the sheet: J6
Changed lines of the file:
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@@
     (stroke (width 0) (type default))
   )
-  (wire (pts (xy 374.396 65.532) (xy 379.476 65.532))
+  (wire (pts (xy 370.713 64.643) (xy 375.793 64.643))
     (stroke (width 0) (type default))
   )
@@
     (stroke (width 0) (type default))
   )
-  (wire (pts (xy 374.396 62.992) (xy 379.476 62.992))
+  (wire (pts (xy 370.713 62.103) (xy 375.793 62.103))
     (stroke (width 0) (type default))
   )
@@
     )
   )
-  (global_label "UART_RX" (shape input) (at 379.476 65.532 0) (fields_autoplaced)
-    (effects (font (size 1.27 1.27)) (justify left))
-    (property "Intersheetrefs" "${INTERSHEET_REFS}" (at 390.565 65.532 0)
+  (global_label "UART_RX" (shape input) (at 375.793 64.643 0) (fields_autoplaced)
+    (effects (font (size 1.27 1.27)) (justify left))
+    (property "Intersheetrefs" "${INTERSHEET_REFS}" (at 386.882 64.643 0)
       (effects (font (size 1.27 1.27)) (justify left) hide)
     )
@@
     )
   )
-  (global_label "UART_TX" (shape input) (at 379.476 62.992 0) (fields_autoplaced)
-    (effects (font (size 1.27 1.27)) (justify left))
-    (property "Intersheetrefs" "${INTERSHEET_REFS}" (at 390.2626 62.992 0)
+  (global_label "UART_TX" (shape input) (at 375.793 62.103 0) (fields_autoplaced)
+    (effects (font (size 1.27 1.27)) (justify left))
+    (property "Intersheetrefs" "${INTERSHEET_REFS}" (at 386.5796 62.103 0)
       (effects (font (size 1.27 1.27)) (justify left) hide)
     )
@@
     )
   )
-  (symbol (lib_id "Connector:Conn_01x02_Pin") (at 369.316 62.992 0) (unit 1)
-    (in_bom yes) (on_board yes) (dnp no) (fields_autoplaced)
-    (property "Reference" "J6" (at 369.951 57.912 0)
-      (effects (font (size 1.27 1.27)))
-    )
-    (property "Value" "Conn_01x02_Pin" (at 369.951 60.452 0)
-      (effects (font (size 1.27 1.27)))
-    )
-    (property "Footprint" "Connector_PinHeader_2.54mm:PinHeader_1x02_P2.54mm_Horizontal" (at 369.316 62.992 0)
-      (effects (font (size 1.27 1.27)) hide)
-    )
-    (property "Datasheet" "~" (at 369.316 62.992 0)
-      (effects (font (size 1.27 1.27)) hide)
-    )
+  (symbol (lib_id "Connector:Conn_01x02_Pin") (at 365.633 62.103 0) (unit 1)
+    (in_bom yes) (on_board yes) (dnp no) (fields_autoplaced)
+    (property "Reference" "J6" (at 366.268 57.023 0)
+      (effects (font (size 1.27 1.27)))
+    )
+    (property "Value" "Conn_01x02_Pin" (at 366.268 59.563 0)
+      (effects (font (size 1.27 1.27)))
+    )
+    (property "Footprint" "Connector_PinHeader_2.54mm:PinHeader_1x02_P2.54mm_Horizontal" (at 365.633 62.103 0)
+      (effects (font (size 1.27 1.27)) hide)
+    )
+    (property "Datasheet" "~" (at 365.633 62.103 0)
+      (effects (font (size 1.27 1.27)) hide)
+    )
