File: HTMDv2.2s.kicad_pcb (KiCad board)
At the start: 2 copper layers, 90 x 55 mm, 46 parts, among them IC2 A3921KLPTR-T, J4 Conn_01x01, J5 Conn_01x01_Pin, J6 Conn_01x02_Pin, J7 Conn_01x01_Pin, J8 Conn_01x01, J9 Conn_01x04_Pin, SW3 SW_Push, U13 SQJ180EP-T1_GE3, U14 SQJ180EP-T1_GE3, U15 SQJ180EP-T1_GE3, U16 SQJ180EP-T1_GE3, U2 STM32F303K8Tx, U3 ISO6741FDWR, U4 CZ3A07

Commit message: update
Parts:
- removed G***: LOGO, 0-Myparts:smallshcale
- added C10: 0.1u, Capacitor_SMD:C_0603_1608Metric_Pad1.08x0.95mm_HandSolder, F.Cu at (215.1, 109.6)
- added C11: 0.1u, Capacitor_SMD:C_0603_1608Metric_Pad1.08x0.95mm_HandSolder, F.Cu at (215.1, 112.1)
- added C12: 4.7u, Capacitor_SMD:C_0603_1608Metric_Pad1.08x0.95mm_HandSolder, F.Cu at (219.4, 92.0)
- added C15: 10u, Capacitor_SMD:C_0805_2012Metric_Pad1.18x1.45mm_HandSolder, F.Cu at (253.3, 101.6)
- added C16: 0.1u, Capacitor_SMD:C_0603_1608Metric_Pad1.08x0.95mm_HandSolder, F.Cu at (219.4, 94.5)
- added C17: 0.1u, Capacitor_SMD:C_0603_1608Metric_Pad1.08x0.95mm_HandSolder, F.Cu at (219.4, 97.0)
- added C18: 0.1u, Capacitor_SMD:C_0603_1608Metric_Pad1.08x0.95mm_HandSolder, F.Cu at (219.4, 99.5)
- added C19: 0.1u, Capacitor_SMD:C_0603_1608Metric_Pad1.08x0.95mm_HandSolder, F.Cu at (219.4, 102.1)
- added C2: 1u, Capacitor_SMD:C_0603_1608Metric_Pad1.08x0.95mm_HandSolder, F.Cu at (215.1, 92.0)
- added C3: 1u, Capacitor_SMD:C_0603_1608Metric_Pad1.08x0.95mm_HandSolder, F.Cu at (215.1, 94.5)
- added C4: 1n, Capacitor_SMD:C_0603_1608Metric_Pad1.08x0.95mm_HandSolder, F.Cu at (215.1, 97.0)
- added C5: 1n, Capacitor_SMD:C_0603_1608Metric_Pad1.08x0.95mm_HandSolder, F.Cu at (215.1, 99.5)
- added C6: 1n, Capacitor_SMD:C_0603_1608Metric_Pad1.08x0.95mm_HandSolder, F.Cu at (215.1, 102.1)
- added C8: 0.1u, Capacitor_SMD:C_0603_1608Metric_Pad1.08x0.95mm_HandSolder, F.Cu at (215.1, 104.6)
- added C9: C, Capacitor_SMD:C_0603_1608Metric_Pad1.08x0.95mm_HandSolder, F.Cu at (215.1, 107.1)
- added J1: Conn_01x04, Connector_JST:JST_XH_S4B-XH-A_1x04_P2.50mm_Horizontal, F.Cu at (233.8, 94.1)
- added J10: Conn_01x02, Connector_JST:JST_XH_S2B-XH-A_1x02_P2.50mm_Horizontal, F.Cu at (235.8, 80.5)
- added J11: Conn_01x02, Connector_JST:JST_XH_S2B-XH-A_1x02_P2.50mm_Horizontal, F.Cu at (245.3, 80.5)
- added J2: Conn_01x04, Connector_JST:JST_XH_S4B-XH-A_1x04_P2.50mm_Horizontal, F.Cu at (233.8, 107.6)
- added J3: Conn_01x06, Connector_JST:JST_XH_S6B-XH-A_1x06_P2.50mm_Horizontal, F.Cu at (216.4, 80.5)
- added JP1: Jumper_2_Open, TestPoint:TestPoint_2Pads_Pitch2.54mm_Drill0.8mm, F.Cu at (246.6, 101.7)
- added JP2: SolderJumper_2_Open, Jumper:SolderJumper-2_P1.3mm_Open_TrianglePad1.0x1.5mm, F.Cu at (246.9, 105.2)
- added JP3: SolderJumper_2_Open, Jumper:SolderJumper-2_P1.3mm_Open_TrianglePad1.0x1.5mm, F.Cu at (246.9, 108.7)
- added JP4: SolderJumper_2_Open, Jumper:SolderJumper-2_P1.3mm_Open_TrianglePad1.0x1.5mm, F.Cu at (246.9, 112.3)
- added JP5: SolderJumper_2_Open, Jumper:SolderJumper-2_P1.3mm_Open_TrianglePad1.0x1.5mm, F.Cu at (246.9, 115.8)
- added R1: 20k, Resistor_SMD:R_0603_1608Metric_Pad0.98x0.95mm_HandSolder, F.Cu at (219.4, 104.6)
- added R10: 120, Resistor_SMD:R_0603_1608Metric, F.Cu at (251.1, 104.7)
- added R17: 10k, Resistor_SMD:R_0603_1608Metric_Pad0.98x0.95mm_HandSolder, F.Cu at (223.8, 102.1)
- added R2: 13k, Resistor_SMD:R_0603_1608Metric_Pad0.98x0.95mm_HandSolder, F.Cu at (219.4, 107.1)
- added R26: 1k, Resistor_SMD:R_0603_1608Metric_Pad0.98x0.95mm_HandSolder, F.Cu at (223.8, 104.6)
- added R27: 1k, Resistor_SMD:R_0603_1608Metric_Pad0.98x0.95mm_HandSolder, F.Cu at (223.8, 107.1)
- added R28: 10k, Resistor_SMD:R_0603_1608Metric_Pad0.98x0.95mm_HandSolder, F.Cu at (223.8, 109.6)
- added R29: 10k, Resistor_SMD:R_0603_1608Metric_Pad0.98x0.95mm_HandSolder, F.Cu at (223.8, 112.1)
- added R3: 2.4k, Resistor_SMD:R_0603_1608Metric_Pad0.98x0.95mm_HandSolder, F.Cu at (219.4, 109.6)
- added R30: 10k, Resistor_SMD:R_0603_1608Metric_Pad0.98x0.95mm_HandSolder, F.Cu at (228.1, 92.0)
- added R31: 13k, Resistor_SMD:R_0603_1608Metric_Pad0.98x0.95mm_HandSolder, F.Cu at (228.1, 94.5)
- added R32: 2.4k, Resistor_SMD:R_0603_1608Metric_Pad0.98x0.95mm_HandSolder, F.Cu at (228.1, 97.0)
- added R4: R, Resistor_SMD:R_0603_1608Metric_Pad0.98x0.95mm_HandSolder, F.Cu at (219.4, 112.1)
- added R5: R, Resistor_SMD:R_0603_1608Metric_Pad0.98x0.95mm_HandSolder, F.Cu at (223.8, 92.0)
- added R6: R, Resistor_SMD:R_0603_1608Metric_Pad0.98x0.95mm_HandSolder, F.Cu at (223.8, 94.5)
- added R8: 20k, Resistor_SMD:R_0603_1608Metric_Pad0.98x0.95mm_HandSolder, F.Cu at (223.8, 97.0)
- added R9: R, Resistor_SMD:R_0603_1608Metric_Pad0.98x0.95mm_HandSolder, F.Cu at (223.8, 99.5)
- added RV1: 10k, Resistor_SMD:R_0603_1608Metric_Pad0.98x0.95mm_HandSolder, F.Cu at (228.1, 99.5)
- added RV2: 10k, Resistor_SMD:R_0603_1608Metric_Pad0.98x0.95mm_HandSolder, F.Cu at (228.1, 102.1)
- added U5: MCP3421A0T-ECH, Package_TO_SOT_SMD:SOT-23-6_Handsoldering, F.Cu at (84.8, 92.8)
- C1: moved to B.Cu
- C7: value C -> 0.1u
- U2: value STM32F303K8Tx -> STM32G431CBUx; footprint Package_QFP:LQFP-32_7x7mm_P0.8mm -> Package_DFN_QFN:QFN-48-1EP_7x7mm_P0.5mm_EP5.6x5.6mm
- moved U3 248.8 mm to (127.5, 69.1)
- moved C13 150.3 mm to (256.4, 19.1)
- moved C21 150.3 mm to (242.1, 18.1)
- moved C27 150.3 mm to (242.1, 15.3)
- moved IC2 150.3 mm to (249.4, 14.1)
- moved R11 150.3 mm to (250.4, 6.08)
- moved R12 150.3 mm to (255.7, 10.3)
- moved R14 150.3 mm to (242.2, 6.23)
- moved R15 150.3 mm to (248.5, 6.08)
- moved R18 150.3 mm to (242.1, 16.6)
- moved R21 150.3 mm to (240.0, 21.4)
- moved R7 150.3 mm to (253.4, 6.89)
- moved SW3 150.3 mm to (245.8, 4.86)
- moved C14 150.3 mm to (255.4, 15.1)
- moved C20 150.3 mm to (257.5, 15.3)
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Connections:
- J9 pad 4: Net-(D4-K) -> +3.3V
- U2 pad 10: LED1 -> OSR1
- U2 pad 11: LED2 -> OPHASE1
- U2 pad 12: ENC_A -> unconnected-(U2-PA4-Pad12)
- U2 pad 13: ENC_B -> SPI_SCK
- U2 pad 14: LED3 -> SPI_MISO
- U2 pad 15: LED4 -> SPI_MOSI
- U2 pad 16: GND -> SPI_CS
- U2 pad 17: +3.3V -> unconnected-(U2-PB0-Pad17)
- U2 pad 18: LED6 -> unconnected-(U2-PB1-Pad18)
- U2 pad 19: UART_TX -> unconnected-(U2-PB2-Pad19)
- U2 pad 20: UART_RX -> +3.3V
- U2 pad 21: CAN_RX -> +3.3V
- U2 pad 22: CAN_TX -> unconnected-(U2-PB10-Pad22)
- U2 pad 23: SWDIO -> +3.3V
- U2 pad 24: SWCLK -> unconnected-(U2-PB11-Pad24)
- U2 pad 25: I2C_SCL -> LED5
- U2 pad 26: SPI_SCK -> LED4
- U2 pad 27: SPI_MISO -> LED3
- U2 pad 28: SPI_MOSI -> LED2
- U2 pad 29: LED5 -> LED1
- U2 pad 3: unconnected-(U2-PF1-Pad3) -> OCD1
- U2 pad 30: I2C_SDA -> ENC_A
- U2 pad 31: unconnected-(U2-BOOT0-Pad31) -> ENC_B
- U2 pad 32: GND -> LED_CAN
- U2 pad 4: Net-(U2-NRST) -> OCD2
- U2 pad 5: +3.3V -> unconnected-(U2-PF0-Pad5)
- U2 pad 6: OPWMH1 -> unconnected-(U2-PF1-Pad6)
- U2 pad 7: OPWML1 -> NRST
- U2 pad 8: OSR1 -> OPWMH1
- U2 pad 9: OPHASE1 -> OPWML1
- U4 pad 12: VOUT -> Net-(U4-VOUT)
Routing:
- net +24V: track 55.1 -> 35.4 mm, vias 1 -> 0
- net Net-(R22-Pad1): track 18.2 -> 5.10 mm, vias 2 -> 1
- net SB1: track 27.9 -> 22.2 mm, vias 2 -> 1
- net Net-(R23-Pad1): track 10.7 -> 5.92 mm, vias 1 -> 0
- net MOSI: track 3.43 -> 0.00 mm
- net LED1: track 2.36 -> 0.00 mm
- net LED2: track 1.68 -> 0.00 mm
- net GNDPWR: vias 49 -> 12
- net GND: vias 29 -> 0
- added copper zone on F.Cu, net (none)

Commit message: update PCB
Parts:
- added D1: D, 0-Myparts:SS2040FL, F.Cu at (217.7, 59.2)
- added IC1: TJA1441AT_0Z, 0-Myparts:SOIC127P600X175-8N, F.Cu at (125.1, 50.9)
- added IC3: TMP275AQDGKRQ1, 0_Mylib:TMP275AQDGKRQ1, F.Cu at (91.3, 64.2)
- added SW2: SW_Push, 0-Myparts:TVAF06, F.Cu at (128.3, 77.3)
- added U1: ADP3338AKCZ-3.3, 0-Myparts:SOT230P700X180-4N, F.Cu at (134.3, 52.9)
- C13, J1, J10, J11, J2, J3: moved to B.Cu
- C7: moved to F.Cu
- RV1, RV2: footprint Resistor_SMD:R_0603_1608Metric_Pad0.98x0.95mm_HandSolder -> 0-Myparts:TSR-3296
- U4: footprint 0_Mylib:CZ3A07 -> 0-Myparts:CZ3AG6
- moved R17 170.6 mm to (90.7, 61.6), turned to 180 degrees
- moved C15 163.2 mm to (91.0, 84.9)
- moved C7 154.4 mm to (113.2, 71.7), turned to -90 degrees
- moved R10 148.1 mm to (113.8, 49.0)
- moved J2 143.2 mm to (105.6, 43.7)
- moved C14 142.7 mm to (121.4, 64.1)
- moved C22 142.7 mm to (108.0, 59.7)
- moved C23 142.7 mm to (109.7, 70.3)
- moved C26 142.7 mm to (108.0, 62.0)
- moved R15 142.7 mm to (114.5, 55.0)
- moved R23 142.7 mm to (108.2, 57.5)
- moved R24 142.7 mm to (108.2, 61.1)
- moved R25 142.7 mm to (108.2, 59.1)
- moved C13 142.7 mm to (122.4, 68.0)
- moved C20 142.7 mm to (123.4, 64.2)
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Connections:
- R17 pad 1: +3.3V -> VCC
- R17 pad 2: Net-(U2-NRST) -> I2C_SCL
Routing:
- net CANH: track 0.00 -> 31.4 mm, vias 0 -> 2
- net OPHASE1: track 0.00 -> 29.9 mm, vias 0 -> 3
- net GNDPWR: track 53.0 -> 24.4 mm, vias 12 -> 5
- net +3.3V: track 0.00 -> 28.6 mm
- net OSR1: track 0.00 -> 26.8 mm, vias 0 -> 2
- net CANL: track 0.00 -> 24.6 mm
- net OPWMH1: track 0.00 -> 22.5 mm, vias 0 -> 3
- net OPWML1: track 0.00 -> 21.5 mm, vias 0 -> 2
- net SPI_SCK: track 0.00 -> 18.7 mm, vias 0 -> 1
- net VCC: track 0.00 -> 18.6 mm, vias 0 -> 1
- net Net-(R23-Pad1): track 5.92 -> 23.7 mm, vias 0 -> 2
- net SPI_CS: track 0.00 -> 14.7 mm
- net Net-(U4-VOUT): track 0.00 -> 14.0 mm
- net Net-(R22-Pad1): track 5.10 -> 15.1 mm, vias 1 -> 2
- net Net-(R19-Pad2): track 12.8 -> 22.3 mm, vias 1 -> 2
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- removed copper zone on B.Cu, net GND
- removed copper zone on F.Cu, net GND

Commit message: update PCB
Parts:
- moved R6 18.6 mm to (112.4, 75.4), turned to 0 degrees
- moved R9 15.9 mm to (112.4, 73.9), turned to 0 degrees
- moved SW2 9.69 mm to (129.9, 86.8)
- moved R5 8.17 mm to (112.4, 77.0)
- moved C10 2.43 mm to (127.8, 65.8)
- moved C8 1.30 mm to (112.4, 78.5), turned to 0 degrees
- moved C16 1.15 mm to (131.3, 78.5), turned to 180 degrees
- moved U1 0.87 mm to (133.8, 52.2)
Routing:
- net NRST: track 0.00 -> 12.6 mm
- net OPWMH1: track 22.5 -> 33.8 mm
- net OPWML1: track 21.5 -> 30.9 mm
- net +24V: track 37.5 -> 32.5 mm
- net OSR1: track 26.8 -> 31.6 mm
- net +5VA: track 36.5 -> 35.8 mm
- net +3.3V: vias 0 -> 2
Other:
- board text added: "Driver RST"
- board text added: "MCU RST"

Commit message: Update HTMDv2.2s.kicad_pcb
Parts:
- removed the R17 at (90.7, 61.6)
- moved R17 141.7 mm to (87.1, 64.6), turned to 90 degrees
- moved R10 4.24 mm to (117.6, 50.9), turned to 180 degrees
- moved C11 0.95 mm to (127.0, 75.1), turned to -90 degrees
Routing:
- net I2C_SCL: track 1.76 -> 39.8 mm, vias 0 -> 2
- net I2C_SDA: track 1.75 -> 36.6 mm, vias 0 -> 2
- net VCC: track 18.6 -> 28.9 mm
- net CANH: track 31.4 -> 34.1 mm
- net +3.3V: track 28.6 -> 29.3 mm
- net Net-(JP1-A): track 2.14 -> 1.97 mm, vias 1 -> 0

Commit message: update
Parts:
- moved JP2 53.9 mm to (175.8, 97.6)
- moved JP3 53.9 mm to (175.8, 100.2)
- moved JP4 53.9 mm to (175.8, 95.0)
- moved R1 53.8 mm to (190.8, 17.3)
- moved R8 53.8 mm to (183.6, 16.9)
- moved J6 31.1 mm to (173.8, 74.7)
- moved J11 27.8 mm to (113.8, 48.8)
- moved J10 27.7 mm to (105.4, 48.8)
- moved C19 25.9 mm to (124.3, 21.5)
- moved C9 25.9 mm to (118.8, 21.5)
- moved IC1 25.9 mm to (120.7, 25.4)
- moved JP1 25.0 mm to (112.3, 24.4)
- moved R10 24.9 mm to (113.5, 26.3)
- moved J1 17.3 mm to (135.7, 48.8)
- moved J2 17.3 mm to (122.2, 48.8)
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Routing:
- net +3.3V: track 29.3 -> 129.0 mm, vias 2 -> 3
- net VCC: track 28.9 -> 127.8 mm, vias 1 -> 4
- net OCD2: track 0.00 -> 66.2 mm, vias 0 -> 2
- net OCD1: track 0.00 -> 63.7 mm, vias 0 -> 2
- net CANH: track 34.1 -> 0.00 mm, vias 2 -> 0
- net SPI_SCK: track 18.7 -> 0.00 mm, vias 1 -> 0
- net SPI_CS: track 14.7 -> 0.49 mm
- net CANL: track 24.6 -> 14.8 mm
- net RESET: track 12.5 -> 17.4 mm
- net NRST: track 12.6 -> 16.3 mm
- net +24V: track 32.5 -> 29.3 mm
- net Net-(JP1-A): track 1.97 -> 0.00 mm
- net OPWML1: track 30.9 -> 32.0 mm
- net GNDPWR: track 24.4 -> 23.4 mm
- net Net-(IC2-RDEAD): track 5.94 -> 5.16 mm
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Other:
- board size 90 x 55 mm -> 90 x 49.9 mm

Commit message: update
配線作業ちう
Parts:
- moved R1 87.1 mm to (126.3, 75.7), turned to -90 degrees
- moved R8 78.3 mm to (127.2, 71.2), turned to 180 degrees
Routing:
- net VREF2: track 2.54 -> 62.8 mm, vias 0 -> 2
- net VREF1: track 2.64 -> 42.9 mm, vias 0 -> 2
- net SPI_SCK: track 0.00 -> 7.98 mm
- net LED_LIM1: track 0.00 -> 6.37 mm
- net GND: track 0.34 -> 4.50 mm
- net LIM1: track 0.00 -> 3.94 mm
- net LIM2: track 0.00 -> 1.77 mm
- net NRST: track 16.3 -> 17.5 mm
- net OPWMH1: track 34.0 -> 34.9 mm

Commit message: Update HTMDv2.2s.kicad_pcb
Parts:
- moved C2 35.5 mm to (179.7, 89.2)
- moved R8 6.45 mm to (126.4, 77.6), turned to -90 degrees
- moved R1 3.70 mm to (129.0, 78.3), turned to 0 degrees
- moved C11 0.05 mm to (129.0, 76.7)
Connections:
- U2 pad 2: unconnected-(U2-PC13-Pad2) -> LED_OCD
Routing:
- net LIM1: track 3.94 -> 50.3 mm
- net LED_LIM1: track 6.37 -> 44.0 mm
- net LIM2: track 1.77 -> 34.0 mm
- net OCD1: track 63.7 -> 65.0 mm
- net OCD2: track 66.2 -> 67.4 mm
- net NRST: track 17.5 -> 18.6 mm
- net OPWMH1: track 34.9 -> 35.6 mm

Commit message: update
update pcb
Parts:
- added REF**: ESD-Logo_13.2x12mm_SilkScreen, Symbol:ESD-Logo_13.2x12mm_SilkScreen, F.Cu at (76.0, 59.3)
- moved R8 47.5 mm to (170.0, 59.0), turned to 90 degrees
- moved C3 16.0 mm to (204.1, 82.8)
- moved C8 12.8 mm to (124.5, 82.4), turned to 180 degrees
- moved C16 11.0 mm to (135.5, 83.2)
- moved SW2 10.9 mm to (138.9, 80.9), turned to 0 degrees
- moved C17 6.59 mm to (94.6, 84.6), turned to 180 degrees
- moved R4 6.12 mm to (115.3, 82.4), turned to 0 degrees
- moved R31 5.85 mm to (131.2, 87.6), turned to 0 degrees
- moved U1 4.82 mm to (137.0, 56.8)
- moved R1 3.71 mm to (126.2, 75.8), turned to -90 degrees
- moved C4 2.17 mm to (119.2, 83.6), turned to 0 degrees
- moved C10 1.98 mm to (129.6, 65.1), turned to 90 degrees
- moved C11 1.49 mm to (127.8, 75.8), turned to -90 degrees
- moved R3 1.48 mm to (123.8, 86.7), turned to 90 degrees
- moved R2 1.22 mm to (111.9, 87.5), turned to 0 degrees
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Routing:
- net GND: track 4.50 -> 86.6 mm, vias 0 -> 2
- net LED_LIM2: track 0.00 -> 32.6 mm
- net UART_RX: track 0.00 -> 12.3 mm
- net UART_TX: track 0.00 -> 11.1 mm
- net SWCLK: track 0.00 -> 6.57 mm
- net SWDIO: track 0.00 -> 5.85 mm
- net NRST: track 18.6 -> 13.3 mm
- net LIM1: track 50.3 -> 46.2 mm
- net VREF2: track 62.8 -> 59.5 mm
- net LED_LIM1: track 44.0 -> 41.6 mm
- net OCD2: track 67.4 -> 68.8 mm, vias 2 -> 4
- net OCD1: track 65.0 -> 66.3 mm, vias 2 -> 4
- net I2C_SCL: track 39.6 -> 40.9 mm
- net OPHASE1: track 29.7 -> 30.9 mm, vias 3 -> 2
- net +3.3V: track 129.2 -> 128.0 mm, vias 3 -> 4
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Other:
- board text added: "!Higi Current Area! Do not touch!"
